File: Gloves Flex PCB.sch (EAGLE design)
At the start: 44 parts, among them X1 USB-MICROB

Commit message: Changes as requested by Hannah from Abu Dhabi
Parts:
- removed JP2: (no value), pinhead:PINHD-2X6/90
- removed U$16: SNAP-PAD_7MM_ROUND, hannahsEagleLib:SNAP-PAD_7MM_ROUND
- added JP3: (no value), pinhead:PINHD-2X8
Connections:
- net GND: now also JP3.1, JP3.11, JP3.13, JP3.15, JP3.3, JP3.5, JP3.7, JP3.9, U$10.SNAPPAD, U$11.SNAPPAD; no longer JP2.10, JP2.12, JP2.2, JP2.4, JP2.6, JP2.8, U$16.SNAPPAD
- net N$14: now also JP3.2; no longer U$10.SNAPPAD
- net N$15: now also JP3.4; no longer U$11.SNAPPAD
- net N$16: now also JP3.6; no longer JP2.1
- net N$18: now also JP3.8; no longer JP2.3
- net N$19: now also JP3.10; no longer JP2.5
- net N$20: now also JP3.12; no longer JP2.7
- net N$21: now also JP3.14; no longer JP2.9
- net N$22: now also JP3.16; no longer JP2.11
Changed lines of the file:
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@@
 <part name="U$22" library="hannahsEagleLib" deviceset="SNAP-PAD_7MM_ROUND" device=""/>
 <part name="U$23" library="hannahsEagleLib" deviceset="SNAP-PAD_7MM_ROUND" device=""/>
-<part name="JP2" library="pinhead" deviceset="PINHD-2X6" device="/90"/>
 <part name="LED1" library="SparkFun-LED" deviceset="LED-TRICOLOR-5050" device="NO_IC"/>
-<part name="U$16" library="hannahsEagleLib" deviceset="SNAP-PAD_7MM_ROUND" device=""/>
 <part name="X1" library="SparkFun" deviceset="USB" device="-MICROB"/>
+<part name="JP3" library="pinhead" deviceset="PINHD-2X8" device=""/>
 </parts>
 <sheets>
@@
 <instance part="U$22" gate="G$1" x="226.06" y="12.7" rot="R90"/>
 <instance part="U$23" gate="G$1" x="266.7" y="12.7" rot="R270"/>
-<instance part="JP2" gate="A" x="127" y="-20.32" rot="R90"/>
 <instance part="LED1" gate="D1" x="203.2" y="5.08" rot="R90"/>
-<instance part="U$16" gate="G$1" x="213.36" y="-99.06" rot="R180"/>
 <instance part="X1" gate="G$1" x="238.76" y="-81.28" rot="R270"/>
+<instance part="JP3" gate="A" x="124.46" y="-17.78" rot="MR270"/>
 </instances>
 <busses>
@@
 <pinref part="U$18" gate="G$1" pin="SNAPPAD"/>
 <wire x1="182.88" y1="-15.24" x2="182.88" y2="-5.08" width="0.1524" layer="91"/>
-<pinref part="JP2" gate="A" pin="12"/>
-<wire x1="134.62" y1="-15.24" x2="182.88" y2="-15.24" width="0.1524" layer="91"/>
-<pinref part="JP2" gate="A" pin="10"/>
+<wire x1="121.92" y1="-15.24" x2="124.46" y2="-15.24" width="0.1524" layer="91"/>
+<wire x1="124.46" y1="-15.24" x2="127" y2="-15.24" width="0.1524" layer="91"/>
+<wire x1="127" y1="-15.24" x2="129.54" y2="-15.24" width="0.1524" layer="91"/>
+<wire x1="129.54" y1="-15.24" x2="132.08" y2="-15.24" width="0.1524" layer="91"/>
 <wire x1="132.08" y1="-15.24" x2="134.62" y2="-15.24" width="0.1524" layer="91"/>
-<pinref part="JP2" gate="A" pin="8"/>
-<wire x1="129.54" y1="-15.24" x2="132.08" y2="-15.24" width="0.1524" layer="91"/>
-<pinref part="JP2" gate="A" pin="6"/>
-<wire x1="127" y1="-15.24" x2="129.54" y2="-15.24" width="0.1524" layer="91"/>
-<pinref part="JP2" gate="A" pin="4"/>
-<wire x1="124.46" y1="-15.24" x2="127" y2="-15.24" width="0.1524" layer="91"/>
-<pinref part="JP2" gate="A" pin="2"/>
-<wire x1="121.92" y1="-15.24" x2="124.46" y2="-15.24" width="0.1524" layer="91"/>
+<wire x1="134.62" y1="-15.24" x2="152.4" y2="-15.24" width="0.1524" layer="91"/>
+<wire x1="152.4" y1="-15.24" x2="182.88" y2="-15.24" width="0.1524" layer="91"/>
 <wire x1="182.88" y1="-5.08" x2="193.04" y2="-5.08" width="0.1524" layer="91"/>
 <wire x1="193.04" y1="-5.08" x2="193.04" y2="20.32" width="0.1524" layer="91"/>
@@
 <wire x1="203.2" y1="20.32" x2="205.74" y2="20.32" width="0.1524" layer="91"/>
 <wire x1="205.74" y1="20.32" x2="215.9" y2="20.32" width="0.1524" layer="91"/>
+<pinref part="JP3" gate="A" pin="5"/>
+<pinref part="JP3" gate="A" pin="7"/>
+<junction x="124.46" y="-15.24"/>
+<pinref part="JP3" gate="A" pin="9"/>
+<junction x="127" y="-15.24"/>
+<pinref part="JP3" gate="A" pin="11"/>
+<junction x="129.54" y="-15.24"/>
+<pinref part="JP3" gate="A" pin="13"/>
+<junction x="132.08" y="-15.24"/>
+<pinref part="JP3" gate="A" pin="15"/>
+<junction x="134.62" y="-15.24"/>
+<pinref part="JP3" gate="A" pin="1"/>
+<wire x1="116.84" y1="-15.24" x2="116.84" y2="-5.08" width="0.1524" layer="91"/>
+<wire x1="116.84" y1="-5.08" x2="119.38" y2="-5.08" width="0.1524" layer="91"/>
+<wire x1="119.38" y1="-5.08" x2="152.4" y2="-5.08" width="0.1524" layer="91"/>
+<wire x1="152.4" y1="-5.08" x2="152.4" y2="-15.24" width="0.1524" layer="91"/>
+<junction x="152.4" y="-15.24"/>
+<pinref part="JP3" gate="A" pin="3"/>
+<wire x1="119.38" y1="-15.24" x2="119.38" y2="-5.08" width="0.1524" layer="91"/>
+<junction x="119.38" y="-5.08"/>
 </segment>
 <segment>
@@
 <wire x1="195.58" y1="-71.12" x2="195.58" y2="-86.36" width="0.1524" layer="91"/>
 <wire x1="228.6" y1="-73.66" x2="228.6" y2="-86.36" width="0.1524" layer="91"/>
-<wire x1="228.6" y1="-86.36" x2="213.36" y2="-86.36" width="0.1524" layer="91"/>
-<pinref part="U$16" gate="G$1" pin="SNAPPAD"/>
-<wire x1="213.36" y1="-86.36" x2="195.58" y2="-86.36" width="0.1524" layer="91"/>
-<junction x="213.36" y="-86.36"/>
+<wire x1="228.6" y1="-86.36" x2="195.58" y2="-86.36" width="0.1524" layer="91"/>
 <pinref part="U$4" gate="G$1" pin="GND"/>
 <wire x1="147.32" y1="-71.12" x2="139.7" y2="-71.12" width="0.1524" layer="91"/>
@@
 <wire x1="238.76" y1="-78.74" x2="238.76" y2="-73.66" width="0.1524" layer="91"/>
 <wire x1="238.76" y1="-73.66" x2="228.6" y2="-73.66" width="0.1524" layer="91"/>
+<pinref part="U$11" gate="G$1" pin="SNAPPAD"/>
+<wire x1="99.06" y1="-10.16" x2="99.06" y2="-88.9" width="0.1524" layer="91"/>
+<wire x1="99.06" y1="-88.9" x2="139.7" y2="-88.9" width="0.1524" layer="91"/>
+<junction x="139.7" y="-88.9"/>
+<pinref part="U$10" gate="G$1" pin="SNAPPAD"/>
+<wire x1="93.98" y1="-10.16" x2="93.98" y2="-88.9" width="0.1524" layer="91"/>
+<wire x1="93.98" y1="-88.9" x2="99.06" y2="-88.9" width="0.1524" layer="91"/>
+<junction x="99.06" y="-88.9"/>
 </segment>
 </net>
@@
 <pinref part="U$4" gate="G$1" pin="IN9"/>
 <pinref part="R8" gate="G$1" pin="2"/>
-<wire x1="147.32" y1="-48.26" x2="93.98" y2="-48.26" width="0.1524" layer="91"/>
-<pinref part="U$10" gate="G$1" pin="SNAPPAD"/>
-<wire x1="93.98" y1="-48.26" x2="45.72" y2="-48.26" width="0.1524" layer="91"/>
-<wire x1="93.98" y1="-10.16" x2="93.98" y2="-48.26" width="0.1524" layer="91"/>
+<wire x1="147.32" y1="-48.26" x2="116.84" y2="-48.26" width="0.1524" layer="91"/>
+<pinref part="JP3" gate="A" pin="2"/>
+<wire x1="116.84" y1="-48.26" x2="45.72" y2="-48.26" width="0.1524" layer="91"/>
+<wire x1="116.84" y1="-48.26" x2="116.84" y2="-22.86" width="0.1524" layer="91"/>
+<junction x="116.84" y="-48.26"/>
 </segment>
 </net>
@@
 <pinref part="R9" gate="G$1" pin="2"/>
 <pinref part="U$4" gate="G$1" pin="IN10"/>
-<wire x1="45.72" y1="-50.8" x2="99.06" y2="-50.8" width="0.1524" layer="91"/>
-<pinref part="U$11" gate="G$1" pin="SNAPPAD"/>
-<wire x1="99.06" y1="-50.8" x2="147.32" y2="-50.8" width="0.1524" layer="91"/>
-<wire x1="99.06" y1="-10.16" x2="99.06" y2="-50.8" width="0.1524" layer="91"/>
+<wire x1="45.72" y1="-50.8" x2="119.38" y2="-50.8" width="0.1524" layer="91"/>
+<pinref part="JP3" gate="A" pin="4"/>
+<wire x1="119.38" y1="-50.8" x2="147.32" y2="-50.8" width="0.1524" layer="91"/>
+<wire x1="119.38" y1="-50.8" x2="119.38" y2="-22.86" width="0.1524" layer="91"/>
+<junction x="119.38" y="-50.8"/>
 </segment>
 </net>
@@
 <wire x1="121.92" y1="-53.34" x2="45.72" y2="-53.34" width="0.1524" layer="91"/>
 <wire x1="121.92" y1="-53.34" x2="121.92" y2="-22.86" width="0.1524" layer="91"/>
-<pinref part="JP2" gate="A" pin="1"/>
+<pinref part="JP3" gate="A" pin="6"/>
 </segment>
 </net>
@@
 <wire x1="124.46" y1="-55.88" x2="147.32" y2="-55.88" width="0.1524" layer="91"/>
 <wire x1="124.46" y1="-22.86" x2="124.46" y2="-55.88" width="0.1524" layer="91"/>
-<pinref part="JP2" gate="A" pin="3"/>
+<pinref part="JP3" gate="A" pin="8"/>
 </segment>
 </net>
@@
 <wire x1="127" y1="-58.42" x2="45.72" y2="-58.42" width="0.1524" layer="91"/>
 <wire x1="127" y1="-58.42" x2="127" y2="-22.86" width="0.1524" layer="91"/>
-<pinref part="JP2" gate="A" pin="5"/>
+<pinref part="JP3" gate="A" pin="10"/>
 </segment>
 </net>
@@
 <wire x1="129.54" y1="-60.96" x2="147.32" y2="-60.96" width="0.1524" layer="91"/>
 <wire x1="129.54" y1="-22.86" x2="129.54" y2="-60.96" width="0.1524" layer="91"/>
-<pinref part="JP2" gate="A" pin="7"/>
+<pinref part="JP3" gate="A" pin="12"/>
 </segment>
 </net>
@@
 <wire x1="132.08" y1="-63.5" x2="45.72" y2="-63.5" width="0.1524" layer="91"/>
 <wire x1="132.08" y1="-63.5" x2="132.08" y2="-22.86" width="0.1524" layer="91"/>
-<pinref part="JP2" gate="A" pin="9"/>
+<pinref part="JP3" gate="A" pin="14"/>
 </segment>
 </net>
@@
 <wire x1="134.62" y1="-66.04" x2="147.32" y2="-66.04" width="0.1524" layer="91"/>
 <wire x1="134.62" y1="-22.86" x2="134.62" y2="-66.04" width="0.1524" layer="91"/>
-<pinref part="JP2" gate="A" pin="11"/>
-</segment>
-</net>
+<pinref part="JP3" gate="A" pin="16"/>
+</segment>
+</net>
